File: hardware/Projects/SRF V2/V2_2 (MAX14870)/sofi_v7_main_rev2_2.sch (EAGLE design)
At the start: 82 parts

Commit message: added GND plane vias to minimize current return paths, modified 2POS_BLOCK lib
Parts:
- BATT, PUMP: value 2POS_BLOCK -> 2POS_BLOCK2POS_BLOCK_NOSTANDS; device 2pos_block_terminal:2POS_BLOCK -> 2pos_block_terminal:2POS_BLOCK2POS_BLOCK_NOSTANDS
Changed lines of the file:
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@@
 <part name="GND47" library="supply1" library_urn="urn:adsk.eagle:library:371" deviceset="GND" device=""/>
 <part name="R32" library="rcl" library_urn="urn:adsk.eagle:library:334" deviceset="R-US_" device="M0805" package3d_urn="urn:adsk.eagle:package:23556/2" value="10K"/>
-<part name="BATT" library="2pos_block_terminal" deviceset="2POS_BLOCK" device=""/>
+<part name="BATT" library="2pos_block_terminal" deviceset="2POS_BLOCK" device="2POS_BLOCK_NOSTANDS" value="2POS_BLOCK2POS_BLOCK_NOSTANDS"/>
 <part name="HALL" library="3pos_block_terminal" deviceset="3POS_TERMINAL" device=""/>
 <part name="U$4" library="8pos_block_terminal" deviceset="8POS_TERMINAL" device=""/>
 <part name="U$5" library="8pos_block_terminal" deviceset="8POS_TERMINAL" device=""/>
-<part name="PUMP" library="2pos_block_terminal" deviceset="2POS_BLOCK" device=""/>
+<part name="PUMP" library="2pos_block_terminal" deviceset="2POS_BLOCK" device="2POS_BLOCK_NOSTANDS" value="2POS_BLOCK2POS_BLOCK_NOSTANDS"/>
 <part name="MAX14870" library="MAX14870" deviceset="MAX14870ETC+T" device=""/>
 <part name="GND39" library="supply1" library_urn="urn:adsk.eagle:library:371" deviceset="GND" device=""/>

Commit message: new motor driver footprints with extended pads, thermals test
Parts:
- DRV8835: value DRV8835DSSRDSS12_P9X2_THERMAL -> DRV8835DSSRDSS12_P9X2_THERMAL_EXTENDED; device DRV8835_ultra_librarian:DRV8835DSSRDSS12_P9X2_THERMAL -> DRV8835_ultra_librarian:DRV8835DSSRDSS12_P9X2_THERMAL_EXTENDED
Changed lines of the file:
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@@
 <part name="R27" library="rcl" library_urn="urn:adsk.eagle:library:334" deviceset="R-US_" device="M0805" package3d_urn="urn:adsk.eagle:package:23556/2" value="6.8K"/>
 <part name="GND31" library="supply1" library_urn="urn:adsk.eagle:library:371" deviceset="GND" device=""/>
-<part name="DRV8835" library="DRV8835_ultra_librarian" deviceset="DRV8835DSSR" device="DSS12_P9X2_THERMAL" value="DRV8835DSSRDSS12_P9X2_THERMAL"/>
+<part name="DRV8835" library="DRV8835_ultra_librarian" deviceset="DRV8835DSSR" device="DSS12_P9X2_THERMAL_EXTENDED" value="DRV8835DSSRDSS12_P9X2_THERMAL_EXTENDED"/>
 <part name="GND34" library="supply1" library_urn="urn:adsk.eagle:library:371" deviceset="GND" device=""/>
 <part name="R31" library="rcl" library_urn="urn:adsk.eagle:library:334" deviceset="R-US_" device="M0805" package3d_urn="urn:adsk.eagle:package:23556/2" value="1.1K"/>

Commit message: extended motor driver pads, removed top thermals on power module thermal vias
Parts:
- DRV8838: value DRV8838DSGTDSG8_P9X1P6_THERMAL -> DRV8838DSGTDSG8_P9X1P6_THERMAL_EXTENDED; device DRV8838:DRV8838DSGTDSG8_P9X1P6_THERMAL -> DRV8838:DRV8838DSGTDSG8_P9X1P6_THERMAL_EXTENDED
Changed lines of the file:
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@@
 <part name="GND32" library="supply1" library_urn="urn:adsk.eagle:library:371" deviceset="GND" device=""/>
 <part name="RPI_HEADER" library="con-lsta" library_urn="urn:adsk.eagle:library:161" deviceset="FE20-2" device="" package3d_urn="urn:adsk.eagle:package:8184/1"/>
-<part name="DRV8838" library="DRV8838" deviceset="DRV8838DSGT" device="DSG8_P9X1P6_THERMAL" value="DRV8838DSGTDSG8_P9X1P6_THERMAL"/>
+<part name="DRV8838" library="DRV8838" deviceset="DRV8838DSGT" device="DSG8_P9X1P6_THERMAL_EXTENDED" value="DRV8838DSGTDSG8_P9X1P6_THERMAL_EXTENDED"/>
 <part name="GND45" library="supply1" library_urn="urn:adsk.eagle:library:371" deviceset="GND" device=""/>
 <part name="C24" library="rcl" library_urn="urn:adsk.eagle:library:334" deviceset="C-EU" device="C0603" package3d_urn="urn:adsk.eagle:package:23616/2" value="0.1 uF"/>
